Commit message: FK
Signed-off-by: Jianliang Shen <shenjianliang@hygon.cn>

File: 1_3D_Model/1_URDF/panther_description/urdf/panther_description.urdf (robot description, URDF)
Before this commit: robot panther_description, 10 links, 9 joints
Links:
- link base_link: geometry collision mesh filename=..//meshes/base_link.STL; visual mesh filename=..//meshes/base_link.STL
- link gripper_1_link: geometry collision mesh filename=..//meshes/gripper_1_link.STL; visual mesh filename=..//meshes/gripper_1_link.STL
- link gripper_2_link: geometry collision mesh filename=..//meshes/gripper_2_link.STL; visual mesh filename=..//meshes/gripper_2_link.STL
- link gripper_centor_link: geometry collision mesh filename=..//meshes/gripper_centor_link.STL; visual mesh filename=..//meshes/gripper_centor_link.STL
- link link1: geometry collision mesh filename=..//meshes/link1.STL; visual mesh filename=..//meshes/link1.STL
- link link2: geometry collision mesh filename=..//meshes/link2.STL; visual mesh filename=..//meshes/link2.STL
- link link3: geometry collision mesh filename=..//meshes/link3.STL; visual mesh filename=..//meshes/link3.STL
- link link4: geometry collision mesh filename=..//meshes/link4.STL; visual mesh filename=..//meshes/link4.STL
- link link5: geometry collision mesh filename=..//meshes/link5.STL; visual mesh filename=..//meshes/link5.STL
- link link6: geometry collision mesh filename=..//meshes/link6.STL; visual mesh filename=..//meshes/link6.STL
